File: Kicad/VacuumSensor.sch (KiCad schematic (older format))
At the start: 38 parts, among them IC1 LM2597MX-ADJ_NOPB, IC2 24PCDFA6D, IC3 INA849DR, IC4 TL071CP, IC5 TL071CP, J1 Screw_Terminal_01x03, J2 Conn_01x02, U1 TL431LP, U2 TL431LP

Commit message: 1.02 update removed the unity gain output op amp and Gain trim pot and replaced it witha  0.1% 665 ohm resistor for the instrumentation amp. simplified the voltage reference and 5v circuits. Added an output Pot to be able to to limit it to 3.3v volts. Added an optional arduino nano v3 and rs232 output. along with a NTC 10k Thermistor for temp compensation calcs.
Parts:
- removed IC5: TL071CP, SamacSys_Parts:DIP794W53P254L959H508Q8N, symbol SamacSys_Parts:TL071CP
- removed J1: Screw_Terminal_01x03, TerminalBlock_Phoenix:TerminalBlock_Phoenix_MKDS-1,5-3_1x03_P5.00mm_Horizontal, symbol Connector:Screw_Terminal_01x03
- removed R3, R7: 10k, Resistor_SMD:R_0603_1608Metric, symbol Device:R_Small_US
- removed R5, R9: 10M, Resistor_SMD:R_0603_1608Metric, symbol Device:R_Small_US
- removed TP2, TP3, TP4, TP5: TestPoint, TestPoint:TestPoint_Pad_2.0x2.0mm, symbol Connector:TestPoint
- removed VoutS1: 20k, Potentiometer_THT:Potentiometer_Bourns_3339P_Vertical, symbol Device:R_POT_US
- added A1: Arduino_Nano_v3.x, Module:Arduino_Nano, symbol MCU_Module:Arduino_Nano_v3.x
- added C10, C9: 0.22uF, Capacitor_THT:CP_Radial_D4.0mm_P1.50mm, symbol Device:CP
- added C11: 0.1uF, Capacitor_THT:CP_Radial_D6.3mm_P2.50mm, symbol Device:CP
- added IC5: SP3220EBEY-L_TR, SOP65P640X120-16N, symbol SamacSys_Parts:SP3220EBEY-L_TR
- added J1: Conn_01x02, Connector_PinHeader_2.54mm:PinHeader_1x02_P2.54mm_Vertical, symbol Connector_Generic:Conn_01x02
- added J3: Screw_Terminal_01x05, TerminalBlock_Phoenix:TerminalBlock_Phoenix_MKDS-1,5-5_1x05_P5.00mm_Horizontal, symbol Connector:Screw_Terminal_01x05
- added R6: 10k, Resistor_SMD:R_0603_1608Metric, symbol Device:R_Small_US
- added RG1: YR1B665RCC, RESAD1550W60L630D230, symbol SamacSys_Parts:YR1B665RCC
- added RT1: NTCSP103JF103FT1S, THRMC1005X55N, symbol SamacSys_Parts:NTCSP103JF103FT1S
- added TP1: TestPoint, TestPoint:TestPoint_Pad_2.0x2.0mm, symbol Connector:TestPoint
- C1, C2: footprint Capacitor_THT:C_Disc_D7.5mm_W4.4mm_P5.00mm -> Capacitor_SMD:C_0805_2012Metric_Pad1.15x1.40mm_HandSolder
- C5: renamed from C4; footprint Capacitor_THT:C_Disc_D7.5mm_W4.4mm_P5.00mm -> Capacitor_SMD:C_0805_2012Metric_Pad1.15x1.40mm_HandSolder
- C8: value 1uF -> 0.22uF; footprint Capacitor_THT:CP_Radial_D5.0mm_P2.00mm -> Capacitor_THT:CP_Radial_D4.0mm_P1.50mm
- OutAdj1: renamed from GAIN1; value 5k -> 1M
- R4: value 10k -> 20k
- renumbered VRef1 to 5VADJ1, C6 to C3, C3 to C4, C5 to C6, R6 to R3, R8 to R5, TP1 to TP2
Connections:
- net +10V: now also A1.30 (VIN); no longer C7.1, IC3.8 (+VS), IC4.7 (VCC+)
- net GND: now also OutAdj1.3, A1.29 (GND), A1.4 (GND), C11.2, IC5.1 (~EN), IC5.14 (GND), J3.1 (Pin_1), RT1.2; no longer C8.2
- net at OutAdj1.1: now also IC3.7 (OUT), A1.19 (A0)
- net at OutAdj1.2: now also J3.3 (Pin_3); no longer IC3.2 (RG_1)
- net at IC3.3 (RG_2): now also RG1.1; no longer OutAdj1.3
- net at IC3.6 (REF), IC4.2 (IN-), IC4.6 (OUT)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: now also A1.20 (A1)
- net +5V: now reaches 5VADJ1.1, R2.2, U1.3 (K)
- net +5V: now also C3.1, C7.1, IC3.8 (+VS), IC4.7 (VCC+), TP1.1
- net at D1.2: now also J3.2 (Pin_2)
- net at U2.1 (REF): now also IC4.3 (IN+), R3.2, U2.3 (K)
- new net: IC3.2 (RG_1), RG1.2
- new net: A1.1 (D1/TX), IC5.11 (T1IN)
- new net: IC5.13 (T1OUT), J3.4 (Pin_4)
- new net: A1.27 (+5V), C11.1, IC5.15 (VCC), IC5.16 (~SHDN), J1.1 (Pin_1), R6.1
- new net: C9.1, IC5.2 (C1+)
- new net: C8.1, IC5.3 (V+)
- new net: C9.2, IC5.4 (C1-)
- new net: C10.1, IC5.5 (C2+)
- new net: C10.2, IC5.6 (C2-)
- new net: C8.2, IC5.7 (V-)
- new net: A1.2 (D0/RX), IC5.8 (R1IN)
- new net: IC5.9 (R1OUT), J3.5 (Pin_5)
- new net: A1.21 (A2), R6.2, RT1.1
- new net: A1.6 (D3), J1.2 (Pin_2), R4.1
- no-connect marks 5 -> 4
Other:
- moved on the sheet: 10VSourceAdj1, 5VADJ1, C1, C2, C3, C4, C5, C6, C7, D1, D2, IC1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
